File: HW/coilDriver_sch.kicad_sch (KiCad schematic)
At the start: 15 parts, among them Q1 AO4892, U3 ACS712xLCTR-05B, U4 ACS712xLCTR-05B, U6 EL7202CS

Commit message: initial commit of SW
Parts:
- R5, R8: value 27 -> 47
Changed lines of the file:
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@@
 			)
 		)
-		(property "Value" "27"
+		(property "Value" "47"
 			(at 193.802 59.69 90)
 			(effects
@@
 			)
 		)
-		(property "Value" "27"
+		(property "Value" "47"
 			(at 193.802 107.95 90)
 			(effects

Commit message: update schematic
Connections:
- net IN_FIRST_COIL renamed IN_COIL0
- net IN_SECOND_COIL renamed IN_COIL1
Changed lines of the file:
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@@
 		)
 	)
-	(hierarchical_label "IN_SECOND_COIL"
+	(hierarchical_label "IN_COIL1"
 		(shape input)
 		(at 83.82 80.01 180)
@@
 		)
 	)
-	(hierarchical_label "IN_FIRST_COIL"
+	(hierarchical_label "IN_COIL0"
 		(shape input)
 		(at 83.82 74.93 180)

Commit message: update HW, reduce board to 5x5 cm
Parts:
- C3, C4: footprint Capacitor_SMD:C_0805_2012Metric_Pad1.18x1.45mm_HandSolder -> Capacitor_SMD:C_1210_3225Metric_Pad1.33x2.70mm_HandSolder
- D1, D2: value SMAJ24CA -> SMBJ24CA; footprint Diode_SMD:D_SMA -> Diode_SMD:D_SMB
- Q1: value AO4892 -> DMTH6016LSD-13
- R3, R4, R6, R7: footprint Capacitor_SMD:C_0603_1608Metric_Pad1.08x0.95mm_HandSolder -> Resistor_SMD:R_0603_1608Metric_Pad0.98x0.95mm_HandSolder
- R5, R8: footprint Capacitor_SMD:C_0805_2012Metric_Pad1.18x1.45mm_HandSolder -> Resistor_SMD:R_1206_3216Metric_Pad1.30x1.75mm_HandSolder
Changed lines of the file:
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@@
 			)
 		)
-		(property "Footprint" "Capacitor_SMD:C_0603_1608Metric_Pad1.08x0.95mm_HandSolder"
+		(property "Footprint" "Resistor_SMD:R_0603_1608Metric_Pad0.98x0.95mm_HandSolder"
 			(at 93.98 86.36 0)
 			(effects
@@
 			)
 		)
-		(property "Footprint" "Capacitor_SMD:C_0805_2012Metric_Pad1.18x1.45mm_HandSolder"
+		(property "Footprint" "Capacitor_SMD:C_1210_3225Metric_Pad1.33x2.70mm_HandSolder"
 			(at 191.77 114.3 0)
 			(effects
@@
 			)
 		)
-		(property "Footprint" "Capacitor_SMD:C_0603_1608Metric_Pad1.08x0.95mm_HandSolder"
+		(property "Footprint" "Resistor_SMD:R_0603_1608Metric_Pad0.98x0.95mm_HandSolder"
 			(at 157.48 107.95 0)
 			(effects
@@
 			)
 		)
-		(property "Value" "AO4892"
+		(property "Value" "DMTH6016LSD-13"
 			(at 177.8 109.2199 0)
 			(effects
@@
 			)
 		)
-		(property "Footprint" "Capacitor_SMD:C_0603_1608Metric_Pad1.08x0.95mm_HandSolder"
+		(property "Footprint" "Resistor_SMD:R_0603_1608Metric_Pad0.98x0.95mm_HandSolder"
 			(at 102.87 86.36 0)
 			(effects
@@
 			)
 		)
-		(property "Value" "AO4892"
+		(property "Value" "DMTH6016LSD-13"
 			(at 177.8 62.2299 0)
 			(effects
@@
 			)
 		)
-		(property "Footprint" "Capacitor_SMD:C_0805_2012Metric_Pad1.18x1.45mm_HandSolder"
+		(property "Footprint" "Resistor_SMD:R_1206_3216Metric_Pad1.30x1.75mm_HandSolder"
 			(at 191.77 59.69 0)
 			(effects
@@
 			)
 		)
-		(property "Footprint" "Capacitor_SMD:C_0805_2012Metric_Pad1.18x1.45mm_HandSolder"
+		(property "Footprint" "Resistor_SMD:R_1206_3216Metric_Pad1.30x1.75mm_HandSolder"
 			(at 191.77 107.95 0)
 			(effects
@@
 			)
 		)
-		(property "Value" "SMAJ24CA"
+		(property "Value" "SMBJ24CA"
 			(at 176.53 49.5299 90)
 			(effects
@@
 			)
 		)
-		(property "Footprint" "Diode_SMD:D_SMA"
+		(property "Footprint" "Diode_SMD:D_SMB"
 			(at 179.07 48.26 0)
 			(effects
@@
 	)
 	(symbol
+		(lib_id "Device:C_Small")
+		(at 191.77 66.04 0)
+		(unit 1)
+		(exclude_from_sim no)
+		(in_bom yes)
+		(on_board yes)
+		(dnp no)
+		(fields_autoplaced yes)
+		(property "Reference" "C3"
+			(at 194.31 64.7762 0)
+			(effects
+				(font
+					(size 1.27 1.27)
+				)
+				(justify left)
+			)
+		)
+		(property "Value" "1µF"
+			(at 194.31 67.3162 0)
+			(effects
+				(font
+					(size 1.27 1.27)
+				)
+				(justify left)
+			)
+		)
+		(property "Footprint" "Capacitor_SMD:C_1210_3225Metric_Pad1.33x2.70mm_HandSolder"
+			(at 191.77 66.04 0)
+			(effects
+				(font
+					(size 1.27 1.27)
+				)
+				(hide yes)
+			)
+		)
+		(property "Datasheet" "~"
+			(at 191.77 66.04 0)
+			(effects
+				(font
+					(size 1.27 1.27)
+				)
+				(hide yes)
+			)
+		)
+		(property "Description" "Unpolarized capacitor, small symbol"
+			(at 191.77 66.04 0)
+			(effects
+				(font
+					(size 1.27 1.27)
+				)
+				(hide yes)
+			)
+		)
+		(pin "1"
+		)
+		(pin "2"
+		)
+		(instances
+			(project "marble_accelerator"
+				(path "/338fb3bb-e550-4c92-aa76-5d93a75fae71/6775c7a4-de2e-4cb3-9e2b-2f99b07eb7c5"
+					(reference "C3")
+					(unit 1)
+				)
+			)
+		)
+	)
+	(symbol
 		(lib_id "Device:R_Small")
 		(at 157.48 60.96 90)
@@
 			)
 		)
-		(property "Footprint" "Capacitor_SMD:C_0603_1608Metric_Pad1.08x0.95mm_HandSolder"
+		(property "Footprint" "Resistor_SMD:R_0603_1608Metric_Pad0.98x0.95mm_HandSolder"
 			(at 157.48 60.96 0)
 			(effects
@@
 			)
 		)
-		(property "Value" "SMAJ24CA"
+		(property "Value" "SMBJ24CA"
 			(at 176.53 97.7899 90)
 			(effects
@@
 			)
 		)
-		(property "Footprint" "Diode_SMD:D_SMA"
+		(property "Footprint" "Diode_SMD:D_SMB"
 			(at 179.07 96.52 0)
 			(effects
@@
 			)
 		)
-		(property "Description" "400W bidirectional Transient Voltage Suppressor, 24.0Vr, SMA(DO-214AC)"
+		(property "Description" "600W bidirectional Transient Voltage Suppressor, 24.0Vr, SMB(DO-214AA)"
 			(at 173.99 96.52 0)
 			(effects
@@
 					(unit 1)
 				)
-			)
-		)
-	)
-	(symbol
-		(lib_id "Device:C_Small")
-		(at 191.77 66.04 0)
-		(unit 1)
-		(exclude_from_sim no)
-		(in_bom yes)
-		(on_board yes)
-		(dnp no)
-		(fields_autoplaced yes)
-		(property "Reference" "C3"
-			(at 194.31 64.7762 0)
-			(effects
-				(font
-					(size 1.27 1.27)
-				)
-				(justify left)
-			)
-		)
-		(property "Value" "1µF"
-			(at 194.31 67.3162 0)
-			(effects
-				(font
-					(size 1.27 1.27)
-				)
-				(justify left)
-			)
-		)
-		(property "Footprint" "Capacitor_SMD:C_0805_2012Metric_Pad1.18x1.45mm_HandSolder"
-			(at 191.77 66.04 0)
-			(effects
-				(font
-					(size 1.27 1.27)
-				)
-				(hide yes)
-			)
-		)
-		(property "Datasheet" "~"
-			(at 191.77 66.04 0)
-			(effects
-				(font
-					(size 1.27 1.27)
-				)
-				(hide yes)
-			)
-		)
-		(property "Description" "Unpolarized capacitor, small symbol"
-			(at 191.77 66.04 0)
-			(effects
-				(font
-					(size 1.27 1.27)
-				)
-				(hide yes)
-			)
-		)
-		(pin "1"
-		)
-		(pin "2"
-		)
-		(instances
-			(project "marble_accelerator"
-				(path "/338fb3bb-e550-4c92-aa76-5d93a75fae71/6775c7a4-de2e-4cb3-9e2b-2f99b07eb7c5"
-					(reference "C3")
-					(unit 1)
-				)

Commit message: update HW
Parts:
- removed U3, U4: ACS712xLCTR-05B, Package_SO:SOIC-8_3.9x4.9mm_P1.27mm, symbol Sensor_Current:ACS712xLCTR-05B
Other:
- moved on the sheet: C3, C4, R5, R8

Commit message: update schematic and board
Parts:
- renumbered C2 to C6, C3 to C7, C4 to C8, D1 to D3, D2 to D4, Q1 to Q2, R5 to R11, R3 to R12, R6 to R13, R7 to R14, R4 to R15, R8 to R16, U6 to U3
Changed lines of the file:
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@@
 		(dnp no)
 		(fields_autoplaced yes)
-		(property "Reference" "R6"
+		(property "Reference" "R13"
 			(at 96.52 85.0899 0)
 			(effects
@@
 			(project "marble_accelerator"
 				(path "/338fb3bb-e550-4c92-aa76-5d93a75fae71/6775c7a4-de2e-4cb3-9e2b-2f99b07eb7c5"
-					(reference "R6")
+					(reference "R13")
 					(unit 1)
 				)
@@
 		(dnp no)
 		(fields_autoplaced yes)
-		(property "Reference" "#PWR03"
+		(property "Reference" "#PWR029"
 			(at 173.99 43.18 0)
 			(effects
@@
 			(project ""
 				(path "/338fb3bb-e550-4c92-aa76-5d93a75fae71/6775c7a4-de2e-4cb3-9e2b-2f99b07eb7c5"
-					(reference "#PWR03")
+					(reference "#PWR029")
 					(unit 1)
 				)
@@
 		(dnp no)
 		(fields_autoplaced yes)
-		(property "Reference" "C4"
+		(property "Reference" "C8"
 			(at 201.93 113.0362 0)
 			(effects
@@
 			(project "marble_accelerator"
 				(path "/338fb3bb-e550-4c92-aa76-5d93a75fae71/6775c7a4-de2e-4cb3-9e2b-2f99b07eb7c5"
-					(reference "C4")
+					(reference "C8")
 					(unit 1)
 				)
@@
 		(dnp no)
 		(fields_autoplaced yes)
-		(property "Reference" "#PWR08"
+		(property "Reference" "#PWR037"
 			(at 121.92 100.33 0)
 			(effects
@@
 			(project "marble_accelerator"
 				(path "/338fb3bb-e550-4c92-aa76-5d93a75fae71/6775c7a4-de2e-4cb3-9e2b-2f99b07eb7c5"
-					(reference "#PWR08")
+					(reference "#PWR037")
 					(unit 1)
 				)
@@
 		(on_board yes)
 		(dnp no)
-		(property "Reference" "R4"
+		(property "Reference" "R15"
 			(at 156.718 105.918 90)
 			(effects
@@
 			(project "marble_accelerator"
 				(path "/338fb3bb-e550-4c92-aa76-5d93a75fae71/6775c7a4-de2e-4cb3-9e2b-2f99b07eb7c5"
-					(reference "R4")
+					(reference "R15")
 					(unit 1)
 				)
@@
 		(dnp no)
 		(fields_autoplaced yes)
-		(property "Reference" "#PWR04"
+		(property "Reference" "#PWR034"
 			(at 173.99 88.9 0)
 			(effects
@@
 			(project ""
 				(path "/338fb3bb-e550-4c92-aa76-5d93a75fae71/6775c7a4-de2e-4cb3-9e2b-2f99b07eb7c5"
-					(reference "#PWR04")
+					(reference "#PWR034")
 					(unit 1)
 				)
@@
 		(dnp no)
 		(fields_autoplaced yes)
-		(property "Reference" "C2"
+		(property "Reference" "C6"
 			(at 113.03 58.4262 0)
 			(effects
@@
 			(project ""
 				(path "/338fb3bb-e550-4c92-aa76-5d93a75fae71/6775c7a4-de2e-4cb3-9e2b-2f99b07eb7c5"
-					(reference "C2")
+					(reference "C6")
 					(unit 1)
 				)
@@
 		(dnp no)
 		(fields_autoplaced yes)
-		(property "Reference" "#PWR011"
+		(property "Reference" "#PWR039"
 			(at 199.39 124.46 0)
 			(effects
@@
 			(project "marble_accelerator"
 				(path "/338fb3bb-e550-4c92-aa76-5d93a75fae71/6775c7a4-de2e-4cb3-9e2b-2f99b07eb7c5"
-					(reference "#PWR011")
+					(reference "#PWR039")
 					(unit 1)
 				)
@@
 		(dnp no)
 		(fields_autoplaced yes)
-		(property "Reference" "#PWR06"
+		(property "Reference" "#PWR038"
 			(at 173.99 124.46 0)
 			(effects
@@
 			(project ""
 				(path "/338fb3bb-e550-4c92-aa76-5d93a75fae71/6775c7a4-de2e-4cb3-9e2b-2f99b07eb7c5"
-					(reference "#PWR06")
+					(reference "#PWR038")
 					(unit 1)
 				)
@@
 		(dnp no)
 		(fields_autoplaced yes)
-		(property "Reference" "Q1"
+		(property "Reference" "Q2"
 			(at 177.8 106.6799 0)
 			(effects
@@
 			(project "marble_accelerator"
 				(path "/338fb3bb-e550-4c92-aa76-5d93a75fae71/6775c7a4-de2e-4cb3-9e2b-2f99b07eb7c5"
-					(reference "Q1")
+					(reference "Q2")
 					(unit 2)
 				)
@@
 		(dnp no)
 		(fields_autoplaced yes)
-		(property "Reference" "#PWR012"
+		(property "Reference" "#PWR035"
 			(at 93.98 100.33 0)
 			(effects
@@
 			(project "marble_accelerator"
 				(path "/338fb3bb-e550-4c92-aa76-5d93a75fae71/6775c7a4-de2e-4cb3-9e2b-2f99b07eb7c5"
-					(reference "#PWR012")
+					(reference "#PWR035")
 					(unit 1)
 				)
@@
 		(dnp no)
 		(fields_autoplaced yes)
-		(property "Reference" "#PWR010"
+		(property "Reference" "#PWR033"
 			(at 199.39 76.2 0)
 			(effects
@@
 			(project "marble_accelerator"
 				(path "/338fb3bb-e550-4c92-aa76-5d93a75fae71/6775c7a4-de2e-4cb3-9e2b-2f99b07eb7c5"
-					(reference "#PWR010")
+					(reference "#PWR033")
 					(unit 1)
 				)
@@
 		(dnp no)
 		(fields_autoplaced yes)
-		(property "Reference" "R7"
+		(property "Reference" "R14"
 			(at 105.41 85.0899 0)
 			(effects
@@
 			(project "marble_accelerator"
 				(path "/338fb3bb-e550-4c92-aa76-5d93a75fae71/6775c7a4-de2e-4cb3-9e2b-2f99b07eb7c5"
-					(reference "R7")
+					(reference "R14")
 					(unit 1)
 				)
@@
 		(dnp no)
 		(fields_autoplaced yes)
-		(property "Reference" "#PWR07"
+		(property "Reference" "#PWR032"
 			(at 173.99 76.2 0)
 			(effects
@@
 			(project ""
 				(path "/338fb3bb-e550-4c92-aa76-5d93a75fae71/6775c7a4-de2e-4cb3-9e2b-2f99b07eb7c5"
-					(reference "#PWR07")
+					(reference "#PWR032")
 					(unit 1)
 				)
@@
 		(dnp no)
 		(fields_autoplaced yes)
-		(property "Reference" "Q1"
+		(property "Reference" "Q2"
 			(at 177.8 59.6899 0)
 			(effects
@@
 			(project "marble_accelerator"
 				(path "/338fb3bb-e550-4c92-aa76-5d93a75fae71/6775c7a4-de2e-4cb3-9e2b-2f99b07eb7c5"
-					(reference "Q1")
+					(reference "Q2")
 					(unit 1)
 				)
@@
 		(dnp no)
 		(fields_autoplaced yes)
-		(property "Reference" "#PWR09"
+		(property "Reference" "#PWR031"
 			(at 110.49 71.12 0)
 			(effects
@@
 			(project ""
 				(path "/338fb3bb-e550-4c92-aa76-5d93a75fae71/6775c7a4-de2e-4cb3-9e2b-2f99b07eb7c5"
-					(reference "#PWR09")
+					(reference "#PWR031")
 					(unit 1)
 				)
@@
 		(dnp no)
 		(fields_autoplaced yes)
-		(property "Reference" "U6"
+		(property "Reference" "U3"
 			(at 124.0633 64.77 0)
 			(effects
@@
 			(project "marble_accelerator"
 				(path "/338fb3bb-e550-4c92-aa76-5d93a75fae71/6775c7a4-de2e-4cb3-9e2b-2f99b07eb7c5"
-					(reference "U6")
+					(reference "U3")
 					(unit 1)
 				)
@@
 		(on_board yes)
 		(dnp no)
-		(property "Reference" "R5"
+		(property "Reference" "R11"
 			(at 197.358 60.452 90)
 			(effects
@@
 			(project "marble_accelerator"
 				(path "/338fb3bb-e550-4c92-aa76-5d93a75fae71/6775c7a4-de2e-4cb3-9e2b-2f99b07eb7c5"
-					(reference "R5")
+					(reference "R11")
 					(unit 1)
 				)
@@
 		(on_board yes)
 		(dnp no)
-		(property "Reference" "R8"
+		(property "Reference" "R16"
 			(at 197.358 108.712 90)
 			(effects
@@
 			(project "marble_accelerator"
 				(path "/338fb3bb-e550-4c92-aa76-5d93a75fae71/6775c7a4-de2e-4cb3-9e2b-2f99b07eb7c5"
-					(reference "R8")
+					(reference "R16")
 					(unit 1)
 				)
@@
 		(dnp no)
 		(fields_autoplaced yes)
-		(property "Reference" "D1"
+		(property "Reference" "D3"
 			(at 176.53 46.9899 90)
 			(effects
@@
 			(project "marble_accelerator"
 				(path "/338fb3bb-e550-4c92-aa76-5d93a75fae71/6775c7a4-de2e-4cb3-9e2b-2f99b07eb7c5"
-					(reference "D1")
+					(reference "D3")
 					(unit 1)
 				)
@@
 		(dnp no)
 		(fields_autoplaced yes)
-		(property "Reference" "C3"
+		(property "Reference" "C7"
 			(at 201.93 64.7762 0)
 			(effects
@@
 			(project "marble_accelerator"
 				(path "/338fb3bb-e550-4c92-aa76-5d93a75fae71/6775c7a4-de2e-4cb3-9e2b-2f99b07eb7c5"
-					(reference "C3")
+					(reference "C7")
 					(unit 1)
 				)
@@
 		(on_board yes)
 		(dnp no)
-		(property "Reference" "R3"
+		(property "Reference" "R12"
 			(at 156.718 58.928 90)
 			(effects
@@
 			(project ""
 				(path "/338fb3bb-e550-4c92-aa76-5d93a75fae71/6775c7a4-de2e-4cb3-9e2b-2f99b07eb7c5"
-					(reference "R3")
+					(reference "R12")
 					(unit 1)
 				)
@@
 		(dnp no)
 		(fields_autoplaced yes)
-		(property "Reference" "D2"
+		(property "Reference" "D4"
 			(at 176.53 95.2499 90)
 			(effects
@@
 			(project "marble_accelerator"
 				(path "/338fb3bb-e550-4c92-aa76-5d93a75fae71/6775c7a4-de2e-4cb3-9e2b-2f99b07eb7c5"
-					(reference "D2")
+					(reference "D4")
 					(unit 1)
 				)
@@
 		(dnp no)
 		(fields_autoplaced yes)
-		(property "Reference" "#PWR05"
+		(property "Reference" "#PWR030"
 			(at 121.92 57.15 0)
 			(effects
@@
 			(project ""
 				(path "/338fb3bb-e550-4c92-aa76-5d93a75fae71/6775c7a4-de2e-4cb3-9e2b-2f99b07eb7c5"
-					(reference "#PWR05")
+					(reference "#PWR030")
 					(unit 1)
 				)
@@
 		(dnp no)
 		(fields_autoplaced yes)
-		(property "Reference" "#PWR013"
+		(property "Reference" "#PWR036"
 			(at 102.87 100.33 0)
 			(effects
@@
 			(project "marble_accelerator"
 				(path "/338fb3bb-e550-4c92-aa76-5d93a75fae71/6775c7a4-de2e-4cb3-9e2b-2f99b07eb7c5"
-					(reference "#PWR013")
-					(unit 1)
-				)
+					(reference "#PWR036")
+					(unit 1)
+				)

Commit message: finished first layout
Parts:
- renumbered C6 to C7, C7 to C8, C8 to C9
Changed lines of the file:
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@@
 		(dnp no)
 		(fields_autoplaced yes)
-		(property "Reference" "#PWR029"
+		(property "Reference" "#PWR030"
 			(at 173.99 43.18 0)
 			(effects
@@
 			(project ""
 				(path "/338fb3bb-e550-4c92-aa76-5d93a75fae71/6775c7a4-de2e-4cb3-9e2b-2f99b07eb7c5"
-					(reference "#PWR029")
+					(reference "#PWR030")
 					(unit 1)
 				)
@@
 		(dnp no)
 		(fields_autoplaced yes)
-		(property "Reference" "C8"
+		(property "Reference" "C9"
 			(at 201.93 113.0362 0)
 			(effects
@@
 			(project "marble_accelerator"
 				(path "/338fb3bb-e550-4c92-aa76-5d93a75fae71/6775c7a4-de2e-4cb3-9e2b-2f99b07eb7c5"
-					(reference "C8")
+					(reference "C9")
 					(unit 1)
 				)
@@
 		(dnp no)
 		(fields_autoplaced yes)
-		(property "Reference" "#PWR037"
+		(property "Reference" "#PWR038"
 			(at 121.92 100.33 0)
 			(effects
@@
 			(project "marble_accelerator"
 				(path "/338fb3bb-e550-4c92-aa76-5d93a75fae71/6775c7a4-de2e-4cb3-9e2b-2f99b07eb7c5"
-					(reference "#PWR037")
+					(reference "#PWR038")
 					(unit 1)
 				)
@@
 		(dnp no)
 		(fields_autoplaced yes)
-		(property "Reference" "#PWR034"
+		(property "Reference" "#PWR035"
 			(at 173.99 88.9 0)
 			(effects
@@
 			(project ""
 				(path "/338fb3bb-e550-4c92-aa76-5d93a75fae71/6775c7a4-de2e-4cb3-9e2b-2f99b07eb7c5"
-					(reference "#PWR034")
+					(reference "#PWR035")
 					(unit 1)
 				)
@@
 		(dnp no)
 		(fields_autoplaced yes)
-		(property "Reference" "C6"
+		(property "Reference" "C7"
 			(at 113.03 58.4262 0)
 			(effects
@@
 			(project ""
 				(path "/338fb3bb-e550-4c92-aa76-5d93a75fae71/6775c7a4-de2e-4cb3-9e2b-2f99b07eb7c5"
-					(reference "C6")
+					(reference "C7")
 					(unit 1)
 				)
@@
 		(dnp no)
 		(fields_autoplaced yes)
-		(property "Reference" "#PWR039"
+		(property "Reference" "#PWR040"
 			(at 199.39 124.46 0)
 			(effects
@@
 			(project "marble_accelerator"
 				(path "/338fb3bb-e550-4c92-aa76-5d93a75fae71/6775c7a4-de2e-4cb3-9e2b-2f99b07eb7c5"
-					(reference "#PWR039")
+					(reference "#PWR040")
 					(unit 1)
 				)
@@
 		(dnp no)
 		(fields_autoplaced yes)
-		(property "Reference" "#PWR038"
+		(property "Reference" "#PWR039"
 			(at 173.99 124.46 0)
 			(effects
@@
 			(project ""
 				(path "/338fb3bb-e550-4c92-aa76-5d93a75fae71/6775c7a4-de2e-4cb3-9e2b-2f99b07eb7c5"
-					(reference "#PWR038")
+					(reference "#PWR039")
 					(unit 1)
 				)
@@
 		(dnp no)
 		(fields_autoplaced yes)
-		(property "Reference" "#PWR035"
+		(property "Reference" "#PWR036"
 			(at 93.98 100.33 0)
 			(effects
@@
 			(project "marble_accelerator"
 				(path "/338fb3bb-e550-4c92-aa76-5d93a75fae71/6775c7a4-de2e-4cb3-9e2b-2f99b07eb7c5"
-					(reference "#PWR035")
+					(reference "#PWR036")
 					(unit 1)
 				)
@@
 		(dnp no)
 		(fields_autoplaced yes)
-		(property "Reference" "#PWR033"
+		(property "Reference" "#PWR034"
 			(at 199.39 76.2 0)
 			(effects
@@
 			(project "marble_accelerator"
 				(path "/338fb3bb-e550-4c92-aa76-5d93a75fae71/6775c7a4-de2e-4cb3-9e2b-2f99b07eb7c5"
-					(reference "#PWR033")
+					(reference "#PWR034")
 					(unit 1)
 				)
@@
 		(dnp no)
 		(fields_autoplaced yes)
-		(property "Reference" "#PWR032"
+		(property "Reference" "#PWR033"
 			(at 173.99 76.2 0)
 			(effects
@@
 			(project ""
 				(path "/338fb3bb-e550-4c92-aa76-5d93a75fae71/6775c7a4-de2e-4cb3-9e2b-2f99b07eb7c5"
-					(reference "#PWR032")
+					(reference "#PWR033")
 					(unit 1)
 				)
@@
 		(dnp no)
 		(fields_autoplaced yes)
-		(property "Reference" "#PWR031"
+		(property "Reference" "#PWR032"
 			(at 110.49 71.12 0)
 			(effects
@@
 			(project ""
 				(path "/338fb3bb-e550-4c92-aa76-5d93a75fae71/6775c7a4-de2e-4cb3-9e2b-2f99b07eb7c5"
-					(reference "#PWR031")
+					(reference "#PWR032")
 					(unit 1)
 				)
@@
 		(dnp no)
 		(fields_autoplaced yes)
-		(property "Reference" "C7"
+		(property "Reference" "C8"
 			(at 201.93 64.7762 0)
 			(effects
@@
 			(project "marble_accelerator"
 				(path "/338fb3bb-e550-4c92-aa76-5d93a75fae71/6775c7a4-de2e-4cb3-9e2b-2f99b07eb7c5"
-					(reference "C7")
+					(reference "C8")
 					(unit 1)
 				)
@@
 		(dnp no)
 		(fields_autoplaced yes)
-		(property "Reference" "#PWR030"
+		(property "Reference" "#PWR031"
 			(at 121.92 57.15 0)
 			(effects
@@
 			(project ""
 				(path "/338fb3bb-e550-4c92-aa76-5d93a75fae71/6775c7a4-de2e-4cb3-9e2b-2f99b07eb7c5"
-					(reference "#PWR030")
+					(reference "#PWR031")
 					(unit 1)
 				)
@@
 		(dnp no)
 		(fields_autoplaced yes)
-		(property "Reference" "#PWR036"
+		(property "Reference" "#PWR037"
 			(at 102.87 100.33 0)
 			(effects
@@
 			(project "marble_accelerator"
 				(path "/338fb3bb-e550-4c92-aa76-5d93a75fae71/6775c7a4-de2e-4cb3-9e2b-2f99b07eb7c5"
-					(reference "#PWR036")
-					(unit 1)
-				)
+					(reference "#PWR037")
+					(unit 1)
+				)
