File: HW/power.kicad_sch (KiCad schematic)
At the start: 8 parts, among them U10 L78L12_SOT89, U8 L78L05_SOT89, U9 MCP1703Ax-500xxMB

Commit message: update HW, reduce board to 5x5 cm
Parts:
- added C13: 100nF, Capacitor_SMD:C_0603_1608Metric_Pad1.08x0.95mm_HandSolder, symbol Device:C_Small
- added D6: LED, LED_SMD:LED_PLCC-2_3.4x3.0mm_KA, symbol Device:LED
- added R15: 10k, Resistor_SMD:R_0603_1608Metric_Pad0.98x0.95mm_HandSolder, symbol Device:R_Small
Connections:
- net +12V: now also C13.1
- net +5V: now also D6.2 (A)
- net GND: now also C13.2, R15.2
- new net: D6.1 (K), R15.1

Commit message: update layout and schematic
Parts:
- removed U9: MCP1703Ax-500xxMB, Package_TO_SOT_SMD:SOT-89-3, symbol Regulator_Linear:MCP1703Ax-500xxMB
- added C14: 100µF/25V, Capacitor_THT:CP_Radial_D6.3mm_P2.50mm, symbol Device:C_Polarized_Small
- added R18: 0R, Resistor_SMD:R_0603_1608Metric_Pad0.98x0.95mm_HandSolder, symbol Device:R_Small
Connections:
- net +12V: now also R18.2
- net +5V: now also C14.1
- net GND: now also C14.2
- net at C1.1, C7.1, D3.1 (K)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: now also R18.1

Commit message: update schematic and board
Parts:
- renumbered C14 to C10, C13 to C11, C8 to C12, C7 to C13, C1 to C14, D3 to D5, R18 to R17, R15 to R18, U10 to U4, U8 to U5
Changed lines of the file:
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@@
 		(dnp no)
 		(fields_autoplaced yes)
-		(property "Reference" "#PWR031"
+		(property "Reference" "#PWR043"
 			(at 115.57 110.49 0)
 			(effects
@@
 			(project "marble_accelerator"
 				(path "/338fb3bb-e550-4c92-aa76-5d93a75fae71/b76a0d8c-a338-4440-bffc-7d4bb77cf8a3"
-					(reference "#PWR031")
+					(reference "#PWR043")
 					(unit 1)
 				)
@@
 		(dnp no)
 		(fields_autoplaced yes)
-		(property "Reference" "D3"
+		(property "Reference" "D5"
 			(at 81.28 80.01 0)
 			(effects
@@
 			(project ""
 				(path "/338fb3bb-e550-4c92-aa76-5d93a75fae71/b76a0d8c-a338-4440-bffc-7d4bb77cf8a3"
-					(reference "D3")
+					(reference "D5")
 					(unit 1)
 				)
@@
 		(dnp no)
 		(fields_autoplaced yes)
-		(property "Reference" "C8"
+		(property "Reference" "C12"
 			(at 148.59 92.7162 0)
 			(effects
@@
 			(project "marble_accelerator"
 				(path "/338fb3bb-e550-4c92-aa76-5d93a75fae71/b76a0d8c-a338-4440-bffc-7d4bb77cf8a3"
-					(reference "C8")
+					(reference "C12")
 					(unit 1)
 				)
@@
 		(dnp no)
 		(fields_autoplaced yes)
-		(property "Reference" "#PWR033"
+		(property "Reference" "#PWR048"
 			(at 175.26 111.76 0)
 			(effects
@@
 			(project "marble_accelerator"
 				(path "/338fb3bb-e550-4c92-aa76-5d93a75fae71/b76a0d8c-a338-4440-bffc-7d4bb77cf8a3"
-					(reference "#PWR033")
+					(reference "#PWR048")
 					(unit 1)
 				)
@@
 		(dnp no)
 		(fields_autoplaced yes)
-		(property "Reference" "C14"
+		(property "Reference" "C10"
 			(at 187.96 90.8938 0)
 			(effects
@@
 			(project ""
 				(path "/338fb3bb-e550-4c92-aa76-5d93a75fae71/b76a0d8c-a338-4440-bffc-7d4bb77cf8a3"
-					(reference "C14")
+					(reference "C10")
 					(unit 1)
 				)
@@
 		(dnp no)
 		(fields_autoplaced yes)
-		(property "Reference" "#PWR030"
+		(property "Reference" "#PWR051"
 			(at 90.17 113.03 0)
 			(effects
@@
 			(project "marble_accelerator"
 				(path "/338fb3bb-e550-4c92-aa76-5d93a75fae71/b76a0d8c-a338-4440-bffc-7d4bb77cf8a3"
-					(reference "#PWR030")
+					(reference "#PWR051")
 					(unit 1)
 				)
@@
 		(dnp no)
 		(fields_autoplaced yes)
-		(property "Reference" "#PWR028"
+		(property "Reference" "#PWR044"
 			(at 129.54 110.49 0)
 			(effects
@@
 			(project "marble_accelerator"
 				(path "/338fb3bb-e550-4c92-aa76-5d93a75fae71/b76a0d8c-a338-4440-bffc-7d4bb77cf8a3"
-					(reference "#PWR028")
+					(reference "#PWR044")
 					(unit 1)
 				)
@@
 		(dnp no)
 		(fields_autoplaced yes)
-		(property "Reference" "#PWR026"
+		(property "Reference" "#PWR041"
 			(at 144.78 81.28 0)
 			(effects
@@
 			(project "marble_accelerator"
 				(path "/338fb3bb-e550-4c92-aa76-5d93a75fae71/b76a0d8c-a338-4440-bffc-7d4bb77cf8a3"
-					(reference "#PWR026")
+					(reference "#PWR041")
 					(unit 1)
 				)
@@
 		(dnp no)
 		(fields_autoplaced yes)
-		(property "Reference" "C13"
+		(property "Reference" "C11"
 			(at 142.24 92.7162 0)
 			(effects
@@
 			(project "marble_accelerator"
 				(path "/338fb3bb-e550-4c92-aa76-5d93a75fae71/b76a0d8c-a338-4440-bffc-7d4bb77cf8a3"
-					(reference "C13")
+					(reference "C11")
 					(unit 1)
 				)
@@
 		(dnp no)
 		(fields_autoplaced yes)
-		(property "Reference" "#PWR027"
+		(property "Reference" "#PWR042"
 			(at 181.61 81.28 0)
 			(effects
@@
 			(project "marble_accelerator"
 				(path "/338fb3bb-e550-4c92-aa76-5d93a75fae71/b76a0d8c-a338-4440-bffc-7d4bb77cf8a3"
-					(reference "#PWR027")
+					(reference "#PWR042")
 					(unit 1)
 				)
@@
 		(dnp no)
 		(fields_autoplaced yes)
-		(property "Reference" "U8"
+		(property "Reference" "U5"
 			(at 161.29 80.01 0)
 			(effects
@@
 			(project ""
 				(path "/338fb3bb-e550-4c92-aa76-5d93a75fae71/b76a0d8c-a338-4440-bffc-7d4bb77cf8a3"
-					(reference "U8")
+					(reference "U5")
 					(unit 1)
 				)
@@
 		(dnp no)
 		(fields_autoplaced yes)
-		(property "Reference" "C1"
+		(property "Reference" "C14"
 			(at 92.71 95.9738 0)
 			(effects
@@
 			(project ""
 				(path "/338fb3bb-e550-4c92-aa76-5d93a75fae71/b76a0d8c-a338-4440-bffc-7d4bb77cf8a3"
-					(reference "C1")
+					(reference "C14")
 					(unit 1)
 				)
@@
 		(dnp no)
 		(fields_autoplaced yes)
-		(property "Reference" "#PWR029"
+		(property "Reference" "#PWR045"
 			(at 161.29 110.49 0)
 			(effects
@@
 			(project "marble_accelerator"
 				(path "/338fb3bb-e550-4c92-aa76-5d93a75fae71/b76a0d8c-a338-4440-bffc-7d4bb77cf8a3"
-					(reference "#PWR029")
+					(reference "#PWR045")
 					(unit 1)
 				)
@@
 		(dnp no)
 		(fields_autoplaced yes)
-		(property "Reference" "#PWR025"
+		(property "Reference" "#PWR040"
 			(at 72.39 81.28 0)
 			(effects
@@
 			(project "marble_accelerator"
 				(path "/338fb3bb-e550-4c92-aa76-5d93a75fae71/b76a0d8c-a338-4440-bffc-7d4bb77cf8a3"
-					(reference "#PWR025")
+					(reference "#PWR040")
 					(unit 1)
 				)
@@
 		(dnp no)
 		(fields_autoplaced yes)
-		(property "Reference" "#PWR032"
+		(property "Reference" "#PWR047"
 			(at 146.05 111.76 0)
 			(effects
@@
 			(project "marble_accelerator"
 				(path "/338fb3bb-e550-4c92-aa76-5d93a75fae71/b76a0d8c-a338-4440-bffc-7d4bb77cf8a3"
-					(reference "#PWR032")
+					(reference "#PWR047")
 					(unit 1)
 				)
@@
 		(dnp no)
 		(fields_autoplaced yes)
-		(property "Reference" "U10"
+		(property "Reference" "U4"
 			(at 129.54 80.01 0)
 			(effects
@@
 			(project ""
 				(path "/338fb3bb-e550-4c92-aa76-5d93a75fae71/b76a0d8c-a338-4440-bffc-7d4bb77cf8a3"
-					(reference "U10")
+					(reference "U4")
 					(unit 1)
 				)
@@
 		(dnp no)
 		(fields_autoplaced yes)
-		(property "Reference" "#PWR048"
+		(property "Reference" "#PWR046"
 			(at 139.7 111.76 0)
 			(effects
@@
 			(project "marble_accelerator"
 				(path "/338fb3bb-e550-4c92-aa76-5d93a75fae71/b76a0d8c-a338-4440-bffc-7d4bb77cf8a3"
-					(reference "#PWR048")
+					(reference "#PWR046")
 					(unit 1)
 				)
@@
 		(dnp no)
 		(fields_autoplaced yes)
-		(property "Reference" "C7"
+		(property "Reference" "C13"
 			(at 118.11 95.2562 0)
 			(effects
@@
 			(project "marble_accelerator"
 				(path "/338fb3bb-e550-4c92-aa76-5d93a75fae71/b76a0d8c-a338-4440-bffc-7d4bb77cf8a3"
-					(reference "C7")
+					(reference "C13")
 					(unit 1)
 				)
@@
 		(dnp no)
 		(fields_autoplaced yes)
-		(property "Reference" "#PWR045"
+		(property "Reference" "#PWR050"
 			(at 199.39 111.76 0)
 			(effects
@@
 			(project "marble_accelerator"
 				(path "/338fb3bb-e550-4c92-aa76-5d93a75fae71/b76a0d8c-a338-4440-bffc-7d4bb77cf8a3"
-					(reference "#PWR045")
+					(reference "#PWR050")
 					(unit 1)
 				)
@@
 		(on_board yes)
 		(dnp no)
-		(property "Reference" "R18"
+		(property "Reference" "R17"
 			(at 128.778 74.168 90)
 			(effects
@@
 			(project "marble_accelerator"
 				(path "/338fb3bb-e550-4c92-aa76-5d93a75fae71/b76a0d8c-a338-4440-bffc-7d4bb77cf8a3"
-					(reference "R18")
+					(reference "R17")
 					(unit 1)
 				)
@@
 		(dnp no)
 		(fields_autoplaced yes)
-		(property "Reference" "R15"
+		(property "Reference" "R18"
 			(at 201.93 90.1699 0)
 			(effects
@@
 			(project "marble_accelerator"
 				(path "/338fb3bb-e550-4c92-aa76-5d93a75fae71/b76a0d8c-a338-4440-bffc-7d4bb77cf8a3"
-					(reference "R15")
+					(reference "R18")
 					(unit 1)
 				)
@@
 		(dnp no)
 		(fields_autoplaced yes)
-		(property "Reference" "#PWR051"
+		(property "Reference" "#PWR049"
 			(at 185.42 111.76 0)
 			(effects
@@
 			(project "marble_accelerator"
 				(path "/338fb3bb-e550-4c92-aa76-5d93a75fae71/b76a0d8c-a338-4440-bffc-7d4bb77cf8a3"
-					(reference "#PWR051")
-					(unit 1)
-				)
+					(reference "#PWR049")
+					(unit 1)
+				)

Commit message: finished first layout
Parts:
- renumbered C9 to C10, C10 to C11, C11 to C12, C12 to C13, C13 to C14, C14 to C15
Changed lines of the file:
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@@
 		(dnp no)
 		(fields_autoplaced yes)
-		(property "Reference" "#PWR043"
+		(property "Reference" "#PWR044"
 			(at 115.57 110.49 0)
 			(effects
@@
 			(project "marble_accelerator"
 				(path "/338fb3bb-e550-4c92-aa76-5d93a75fae71/b76a0d8c-a338-4440-bffc-7d4bb77cf8a3"
-					(reference "#PWR043")
+					(reference "#PWR044")
 					(unit 1)
 				)
@@
 		(dnp no)
 		(fields_autoplaced yes)
-		(property "Reference" "C9"
+		(property "Reference" "C10"
 			(at 177.8 91.4462 0)
 			(effects
@@
 			(project "marble_accelerator"
 				(path "/338fb3bb-e550-4c92-aa76-5d93a75fae71/b76a0d8c-a338-4440-bffc-7d4bb77cf8a3"
-					(reference "C9")
+					(reference "C10")
 					(unit 1)
 				)
@@
 		(dnp no)
 		(fields_autoplaced yes)
-		(property "Reference" "C12"
+		(property "Reference" "C13"
 			(at 148.59 92.7162 0)
 			(effects
@@
 			(project "marble_accelerator"
 				(path "/338fb3bb-e550-4c92-aa76-5d93a75fae71/b76a0d8c-a338-4440-bffc-7d4bb77cf8a3"
-					(reference "C12")
+					(reference "C13")
 					(unit 1)
 				)
@@
 		(dnp no)
 		(fields_autoplaced yes)
-		(property "Reference" "#PWR048"
+		(property "Reference" "#PWR049"
 			(at 175.26 111.76 0)
 			(effects
@@
 			(project "marble_accelerator"
 				(path "/338fb3bb-e550-4c92-aa76-5d93a75fae71/b76a0d8c-a338-4440-bffc-7d4bb77cf8a3"
-					(reference "#PWR048")
+					(reference "#PWR049")
 					(unit 1)
 				)
@@
 		(dnp no)
 		(fields_autoplaced yes)
-		(property "Reference" "C10"
+		(property "Reference" "C11"
 			(at 187.96 90.8938 0)
 			(effects
@@
 			(project ""
 				(path "/338fb3bb-e550-4c92-aa76-5d93a75fae71/b76a0d8c-a338-4440-bffc-7d4bb77cf8a3"
-					(reference "C10")
+					(reference "C11")
 					(unit 1)
 				)
@@
 		(dnp no)
 		(fields_autoplaced yes)
-		(property "Reference" "#PWR051"
+		(property "Reference" "#PWR052"
 			(at 90.17 113.03 0)
 			(effects
@@
 			(project "marble_accelerator"
 				(path "/338fb3bb-e550-4c92-aa76-5d93a75fae71/b76a0d8c-a338-4440-bffc-7d4bb77cf8a3"
-					(reference "#PWR051")
+					(reference "#PWR052")
 					(unit 1)
 				)
@@
 		(dnp no)
 		(fields_autoplaced yes)
-		(property "Reference" "#PWR044"
+		(property "Reference" "#PWR045"
 			(at 129.54 110.49 0)
 			(effects
@@
 			(project "marble_accelerator"
 				(path "/338fb3bb-e550-4c92-aa76-5d93a75fae71/b76a0d8c-a338-4440-bffc-7d4bb77cf8a3"
-					(reference "#PWR044")
+					(reference "#PWR045")
 					(unit 1)
 				)
@@
 		(dnp no)
 		(fields_autoplaced yes)
-		(property "Reference" "#PWR041"
+		(property "Reference" "#PWR042"
 			(at 144.78 81.28 0)
 			(effects
@@
 			(project "marble_accelerator"
 				(path "/338fb3bb-e550-4c92-aa76-5d93a75fae71/b76a0d8c-a338-4440-bffc-7d4bb77cf8a3"
-					(reference "#PWR041")
+					(reference "#PWR042")
 					(unit 1)
 				)
@@
 		(dnp no)
 		(fields_autoplaced yes)
-		(property "Reference" "C11"
+		(property "Reference" "C12"
 			(at 142.24 92.7162 0)
 			(effects
@@
 			(project "marble_accelerator"
 				(path "/338fb3bb-e550-4c92-aa76-5d93a75fae71/b76a0d8c-a338-4440-bffc-7d4bb77cf8a3"
-					(reference "C11")
+					(reference "C12")
 					(unit 1)
 				)
@@
 		(dnp no)
 		(fields_autoplaced yes)
-		(property "Reference" "#PWR042"
+		(property "Reference" "#PWR043"
 			(at 181.61 81.28 0)
 			(effects
@@
 			(project "marble_accelerator"
 				(path "/338fb3bb-e550-4c92-aa76-5d93a75fae71/b76a0d8c-a338-4440-bffc-7d4bb77cf8a3"
-					(reference "#PWR042")
+					(reference "#PWR043")
 					(unit 1)
 				)
@@
 		(dnp no)
 		(fields_autoplaced yes)
-		(property "Reference" "C14"
+		(property "Reference" "C15"
 			(at 92.71 95.9738 0)
 			(effects
@@
 			(project ""
 				(path "/338fb3bb-e550-4c92-aa76-5d93a75fae71/b76a0d8c-a338-4440-bffc-7d4bb77cf8a3"
-					(reference "C14")
+					(reference "C15")
 					(unit 1)
 				)
@@
 		(dnp no)
 		(fields_autoplaced yes)
-		(property "Reference" "#PWR045"
+		(property "Reference" "#PWR046"
 			(at 161.29 110.49 0)
 			(effects
@@
 			(project "marble_accelerator"
 				(path "/338fb3bb-e550-4c92-aa76-5d93a75fae71/b76a0d8c-a338-4440-bffc-7d4bb77cf8a3"
-					(reference "#PWR045")
+					(reference "#PWR046")
 					(unit 1)
 				)
@@
 		(dnp no)
 		(fields_autoplaced yes)
-		(property "Reference" "#PWR040"
+		(property "Reference" "#PWR041"
 			(at 72.39 81.28 0)
 			(effects
@@
 			(project "marble_accelerator"
 				(path "/338fb3bb-e550-4c92-aa76-5d93a75fae71/b76a0d8c-a338-4440-bffc-7d4bb77cf8a3"
-					(reference "#PWR040")
+					(reference "#PWR041")
 					(unit 1)
 				)
@@
 		(dnp no)
 		(fields_autoplaced yes)
-		(property "Reference" "#PWR047"
+		(property "Reference" "#PWR048"
 			(at 146.05 111.76 0)
 			(effects
@@
 			(project "marble_accelerator"
 				(path "/338fb3bb-e550-4c92-aa76-5d93a75fae71/b76a0d8c-a338-4440-bffc-7d4bb77cf8a3"
-					(reference "#PWR047")
+					(reference "#PWR048")
 					(unit 1)
 				)
@@
 		(dnp no)
 		(fields_autoplaced yes)
-		(property "Reference" "#PWR046"
+		(property "Reference" "#PWR047"
 			(at 139.7 111.76 0)
 			(effects
@@
 			(project "marble_accelerator"
 				(path "/338fb3bb-e550-4c92-aa76-5d93a75fae71/b76a0d8c-a338-4440-bffc-7d4bb77cf8a3"
-					(reference "#PWR046")
+					(reference "#PWR047")
 					(unit 1)
 				)
@@
 		(dnp no)
 		(fields_autoplaced yes)
-		(property "Reference" "C13"
+		(property "Reference" "C14"
 			(at 118.11 95.2562 0)
 			(effects
@@
 			(project "marble_accelerator"
 				(path "/338fb3bb-e550-4c92-aa76-5d93a75fae71/b76a0d8c-a338-4440-bffc-7d4bb77cf8a3"
-					(reference "C13")
+					(reference "C14")
 					(unit 1)
 				)
@@
 		(dnp no)
 		(fields_autoplaced yes)
-		(property "Reference" "#PWR050"
+		(property "Reference" "#PWR051"
 			(at 199.39 111.76 0)
 			(effects
@@
 			(project "marble_accelerator"
 				(path "/338fb3bb-e550-4c92-aa76-5d93a75fae71/b76a0d8c-a338-4440-bffc-7d4bb77cf8a3"
-					(reference "#PWR050")
+					(reference "#PWR051")
 					(unit 1)
 				)
@@
 		(dnp no)
 		(fields_autoplaced yes)
-		(property "Reference" "#PWR049"
+		(property "Reference" "#PWR050"
 			(at 185.42 111.76 0)
 			(effects
@@
 			(project "marble_accelerator"
 				(path "/338fb3bb-e550-4c92-aa76-5d93a75fae71/b76a0d8c-a338-4440-bffc-7d4bb77cf8a3"
-					(reference "#PWR049")
-					(unit 1)
-				)
+					(reference "#PWR050")
+					(unit 1)
+				)
