File: HW/marble_accelerator.kicad_pcb (KiCad board)
At the start: 2 copper layers, 50 x 50 mm, 62 parts, among them J1 Conn_01x02_Pin, J2 Conn_01x02_Pin, J3 Conn_01x03_Pin, J4 Conn_01x02_Pin, J5 Conn_01x03_Pin, J6 UART, J7 AVR-ISP-6, Q1 BSS138, Q2 DMTH6016LSD-13, U1 CNY70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

Commit message: cosmetic changes on layout
Routing:
- net Net-(D1-A): track 36.9 -> 32.7 mm, vias 2 -> 0
- net /microcontroller/EntryEnable: track 22.2 -> 20.3 mm
Other:
- board text added: "HS"
- board text added: "Marble Accelerator V1.0 03/25"
Changed lines of the file:
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@@
 		(tags "capacitor handsolder")
 		(property "Reference" "C2"
-			(at 2.4 0 0)
+			(at 2.3 0 0)
 			(layer "F.SilkS")
 			(effects
@@
 		(tags "capacitor handsolder")
 		(property "Reference" "C4"
-			(at 0 -1 0)
+			(at 0 -1.1 0)
 			(layer "F.SilkS")
 			(effects
@@
 		(tags "capacitor handsolder")
 		(property "Reference" "C13"
-			(at -0.7 1.8 0)
+			(at -0.9 1.6 0)
 			(layer "F.SilkS")
 			(effects
@@
 		(tags "Through hole pin header THT 1x04 2.54mm single row")
 		(property "Reference" "J6"
-			(at 0 -2.33 0)
+			(at -2.8 4.2 0)
 			(layer "F.SilkS")
 			(effects
@@
 		(property "Value" "UART"
 			(at 0 9.95 0)
-			(layer "F.Fab")
+			(layer "F.SilkS")
 			(effects
 				(font
@@
 		(tags "capacitor handsolder")
 		(property "Reference" "C3"
-			(at 2.4 -0.1 0)
+			(at 2.3 -0.1 0)
 			(layer "F.SilkS")
 			(effects
@@
 		(tags "capacitor handsolder")
 		(property "Reference" "C14"
-			(at -0.7 -1.9 180)
+			(at -0.2 -1.6 180)
 			(layer "F.SilkS")
 			(effects
@@
 		(layer "Edge.Cuts")
 	)
+	(gr_text "HS"
+		(at 149.8 89.6 0)
+		(layer "B.Cu")
+		(effects
+			(font
+				(size 1 1)
+				(thickness 0.1)
+			)
+			(justify left bottom mirror)
+		)
+	)
+	(gr_text "Marble Accelerator V1.0 03/25"
+		(at 125 41.7 0)
+		(layer "B.Cu")
+		(effects
+			(font
+				(size 1 1)
+				(thickness 0.1)
+			)
+			(justify bottom mirror)
+		)
+	)
 	(gr_text "-"
 		(at 140.9 82.1 0)
@@
 	)
 	(segment
-		(start 127.4 59.85)
-		(end 127.4 55.634314)
+		(start 124.609032 45.3615)
+		(end 124.407032 45.5635)
 		(width 0.2)
 		(layer "F.Cu")
@@
 	)
 	(segment
-		(start 128.6 43.6)
-		(end 128.6 41.7)
+		(start 125.357032 45.3615)
+		(end 124.609032 45.3615)
 		(width 0.2)
 		(layer "F.Cu")
@@
 	)
 	(segment
-		(start 127.4 55.634314)
-		(end 129.3 53.734314)
+		(start 129.301 53.233315)
+		(end 129.301 48.401)
 		(width 0.2)
 		(layer "F.Cu")
@@
 	)
 	(segment
-		(start 129.301 53.233315)
-		(end 129.301 46.001)
+		(start 125.559032 45.5635)
+		(end 125.357032 45.3615)
 		(width 0.2)
 		(layer "F.Cu")
@@
 	)
 	(segment
-		(start 129.301 46.001)
-		(end 128.6 45.3)
+		(start 119.3 41.6)
+		(end 113.4 41.6)
 		(width 0.2)
 		(layer "F.Cu")
@@
 	)
 	(segment
-		(start 129.3 53.234315)
-		(end 129.301 53.233315)
+		(start 129.301 48.401)
+		(end 126.4635 45.5635)
+		(width 0.2)
+		(layer "F.Cu")
+		(net 21)
+	)
+	(segment
+		(start 113.4 41.6)
+		(end 113 42)
 		(width 0.2)
 		(layer "F.Cu")
@@
 	)
 	(segment
-		(start 114.4 40.6)
-		(end 113 42)
+		(start 127.4 55.634314)
+		(end 129.3 53.734314)
 		(width 0.2)
 		(layer "F.Cu")
@@
 	)
 	(segment
-		(start 127.5 40.6)
-		(end 114.4 40.6)
+		(start 127.4 59.85)
+		(end 127.4 55.634314)
 		(width 0.2)
 		(layer "F.Cu")
@@
 	)
 	(segment
-		(start 128.6 41.7)
-		(end 127.5 40.6)
+		(start 126.4635 45.5635)
+		(end 125.559032 45.5635)
 		(width 0.2)
 		(layer "F.Cu")
 		(net 21)
 	)
-	(via
-		(at 128.6 45.3)
-		(size 0.6)
-		(drill 0.3)
-		(layers "F.Cu" "B.Cu")
+	(segment
+		(start 129.3 53.234315)
+		(end 129.301 53.233315)
+		(width 0.2)
+		(layer "F.Cu")
 		(net 21)
 	)
-	(via
-		(at 128.6 43.6)
-		(size 0.6)
-		(drill 0.3)
-		(layers "F.Cu" "B.Cu")
+	(segment
+		(start 123.2635 45.5635)
+		(end 119.3 41.6)
+		(width 0.2)
+		(layer "F.Cu")
 		(net 21)
 	)
 	(segment
-		(start 128.6 45.3)
-		(end 128.6 43.6)
+		(start 124.407032 45.5635)
+		(end 123.2635 45.5635)
 		(width 0.2)
-		(layer "B.Cu")
+		(layer "F.Cu")
 		(net 21)
 	)
@@
 	(segment
 		(start 129.700999 54.399001)
-		(end 129.700999 45.100999)
+		(end 129.700999 47.6)
 		(width 0.2)
 		(layer "F.Cu")
@@
 	(segment
 		(start 125.75 44.525)
-		(end 129.125 44.525)
+		(end 126.8 44.525)
 		(width 0.2)
 		(layer "F.Cu")
@@
 	)
 	(segment
-		(start 129.2 44.6)
-		(end 129.562499 44.962499)
+		(start 129.700999 47.425999)
+		(end 129.700999 47.6)
 		(width 0.2)
 		(layer "F.Cu")
@@
 	)
 	(segment
-		(start 129.125 44.525)
-		(end 129.2 44.6)
+		(start 126.8 44.525)
+		(end 129.700999 47.425999)
 		(width 0.2)
 		(layer "F.Cu")
@@
 	)
 	(segment
-		(start 129.700999 45.100999)
-		(end 129.2 44.6)
-		(width 0.2)
-		(layer "F.Cu")
-		(net 22)
-	)
-	(segment
-		(start 121.2 45.4)
-		(end 121.2 43.5)
+		(start 126.6 59.85)
+		(end 126.6 55.75705)
 		(width 0.2)
 		(layer "F.Cu")
@@
 	)
 	(segment
-		(start 128.9 53.45705)
-		(end 128.9 52.4)
+		(start 123.8 48)
+		(end 121.2 45.4)
 		(width 0.2)
 		(layer "F.Cu")
@@
 	)
 	(segment
-		(start 116.8 43)
-		(end 120.7 43)
+		(start 128.3 51.8)
+		(end 124.2 51.8)
 		(width 0.2)
 		(layer "F.Cu")
@@
 	)
 	(segment
-		(start 123.8 48)
-		(end 121.2 45.4)
+		(start 126.6 55.75705)
+		(end 128.9 53.45705)
 		(width 0.2)
 		(layer "F.Cu")
@@
 	)
 	(segment
-		(start 120.7 43)
-		(end 121.2 43.5)
+		(start 128.9 53.45705)
+		(end 128.9 52.4)
 		(width 0.2)
 		(layer "F.Cu")
@@
 	)
 	(segment
-		(start 128.3 51.8)
-		(end 124.2 51.8)
+		(start 120.134314 43)
+		(end 116.8 43)
 		(width 0.2)
 		(layer "F.Cu")
@@
 	)
 	(segment
-		(start 124.2 51.8)
-		(end 123.8 51.4)
+		(start 121.2 45.4)
+		(end 121.2 44.065686)
 		(width 0.2)
 		(layer "F.Cu")
@@
 	)
 	(segment
-		(start 126.6 59.85)
-		(end 126.6 55.75705)
+		(start 124.2 51.8)
+		(end 123.8 51.4)
 		(width 0.2)
 		(layer "F.Cu")
@@
 	)
 	(segment
-		(start 126.6 55.75705)
-		(end 128.9 53.45705)
+		(start 128.9 52.4)
+		(end 128.3 51.8)
 		(width 0.2)
 		(layer "F.Cu")
@@
 	)
 	(segment
-		(start 128.9 52.4)
-		(end 128.3 51.8)
+		(start 121.2 44.065686)
+		(end 120.134314 43)
 		(width 0.2)
 		(layer "F.Cu")
